Commit message: ROS1 and ROS2, Tug robot updates

File: doozy_ws/src/amr_bot/urdf/amr_bot.urdf (robot description, URDF)
Before this commit: robot amr_bot, 8 links, 7 joints
Joints:
- joint base_joint: origin xyz=0.40456 -0.53802 0.48728 rpy=1.5708 0 0 -> xyz=0.40456 -0.53802 0.5 rpy=0 0 0
- joint l_wheel_joint: axis 0 -1 0 -> 0 1 0
- joint sickcam_joint: origin xyz=-0.77559 0.0013357 0.60934 rpy=0 0 0 -> xyz=-0.77559 0.0013357 0.60934 rpy=0 0 3.14
